File: solar_cooker.kicad_pcb (KiCad board)
At the start: 2 copper layers, 152.7 x 77.2 mm, 20 parts, among them J1 Pt100, J2 microSD, J3 clock, J4 Pt100, J5 BME680, J6 GPS, J7 Pt100, J8 display, U1 anemometer, U2 AM2315C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

Commit message: silkscreen update
Parts:
- added G***: LOGO, custom_components:logo, B.Cu at (86.2, 84.1)
Other:
- board text added: "solar cooker testing station v2.2"
- board text removed: "J10"
- board text removed: "J11"
- board text removed: "J12"
- board text removed: "J13"
- board text removed: "J14"
- board text removed: "J15"
- board text removed: "J16"
- board text removed: "J9"
- board text removed: "solar cooker testing station v2.1"
